Commit message: add realsense camera to urdf

File: src/sprayer_description/urdf/sprayer.urdf.xacro (robot description, xacro)
@@ -6,4 +6,5 @@
   name="sprayerAssy2"
   xmlns:xacro="http://ros.org/wiki/xacro">
+  <xacro:include filename="$(find realsense2_description)/urdf/_d435.urdf.xacro" />
   <link
     name="sprayer_base">
@@ -177,3 +178,6 @@
       xyz="0 0 0" />
   </joint>
+  <xacro:sensor_d435 parent="camera_screw" name="camera" use_nominal_extrinsics="true">
+    <origin xyz="0 0 0" rpy="0 0 0"/>
+  </xacro:sensor_d435>
 </robot>

Commit message: switch nozzle frame numbering to 0-based in urdf
easier to work with in code

File: src/sprayer_description/urdf/sprayer.urdf.xacro (robot description, xacro)
@@ -83,4 +83,20 @@
   </joint>
   <link
+    name="spot_nozzle0">
+  </link>
+  <joint
+    name="spot_nozzle0_j"
+    type="fixed">
+    <origin
+      xyz="0 -0.0665988000000001 -0.28575"
+      rpy="1.5707963267949 0 0" />
+    <parent
+      link="spot_boom" />
+    <child
+      link="spot_nozzle0" />
+    <axis
+      xyz="0 0 0" />
+  </joint>
+  <link
     name="spot_nozzle1">
   </link>
@@ -89,5 +105,5 @@
     type="fixed">
     <origin
-      xyz="0 -0.0665988000000001 -0.28575"
+      xyz="0 -0.0665988000000001 -0.09525"
       rpy="1.5707963267949 0 0" />
     <parent
@@ -105,5 +121,5 @@
     type="fixed">
     <origin
-      xyz="0 -0.0665988000000001 -0.09525"
+      xyz="0 -0.0665988000000001 0.09525"
       rpy="1.5707963267949 0 0" />
     <parent
@@ -121,5 +137,5 @@
     type="fixed">
     <origin
-      xyz="0 -0.0665988000000001 0.09525"
+      xyz="0 -0.0665988000000001 0.28575"
       rpy="1.5707963267949 0 0" />
     <parent
@@ -131,24 +147,8 @@
   </joint>
   <link
-    name="spot_nozzle4">
+    name="broadcast_nozzle0">
   </link>
   <joint
-    name="spot_nozzle4_j"
-    type="fixed">
-    <origin
-      xyz="0 -0.0665988000000001 0.28575"
-      rpy="1.5707963267949 0 0" />
-    <parent
-      link="spot_boom" />
-    <child
-      link="spot_nozzle4" />
-    <axis
-      xyz="0 0 0" />
-  </joint>
-  <link
-    name="broadcast_nozzle1">
-  </link>
-  <joint
-    name="broadcast_nozzle1_j"
+    name="broadcast_nozzle0_j"
     type="fixed">
     <origin
@@ -158,5 +158,5 @@
       link="sprayer_base" />
     <child
-      link="broadcast_nozzle1" />
+      link="broadcast_nozzle0" />
     <axis
       xyz="0 0 0" />

Commit message: flip nozzle indices in urdf
aligns with the numbering used by robot wiring/Arduino

File: src/sprayer_description/urdf/sprayer.urdf.xacro (robot description, xacro)
@@ -83,8 +83,8 @@
   </joint>
   <link
-    name="spot_nozzle0">
+    name="spot_nozzle3">
   </link>
   <joint
-    name="spot_nozzle0_j"
+    name="spot_nozzle3_j"
     type="fixed">
     <origin
@@ -94,5 +94,21 @@
       link="spot_boom" />
     <child
-      link="spot_nozzle0" />
+      link="spot_nozzle3" />
+    <axis
+      xyz="0 0 0" />
+  </joint>
+  <link
+    name="spot_nozzle2">
+  </link>
+  <joint
+    name="spot_nozzle2_j"
+    type="fixed">
+    <origin
+      xyz="0 -0.0665988000000001 -0.09525"
+      rpy="1.5707963267949 0 0" />
+    <parent
+      link="spot_boom" />
+    <child
+      link="spot_nozzle2" />
     <axis
       xyz="0 0 0" />
@@ -105,5 +121,5 @@
     type="fixed">
     <origin
-      xyz="0 -0.0665988000000001 -0.09525"
+      xyz="0 -0.0665988000000001 0.09525"
       rpy="1.5707963267949 0 0" />
     <parent
@@ -115,24 +131,8 @@
   </joint>
   <link
-    name="spot_nozzle2">
+    name="spot_nozzle0">
   </link>
   <joint
-    name="spot_nozzle2_j"
-    type="fixed">
-    <origin
-      xyz="0 -0.0665988000000001 0.09525"
-      rpy="1.5707963267949 0 0" />
-    <parent
-      link="spot_boom" />
-    <child
-      link="spot_nozzle2" />
-    <axis
-      xyz="0 0 0" />
-  </joint>
-  <link
-    name="spot_nozzle3">
-  </link>
-  <joint
-    name="spot_nozzle3_j"
+    name="spot_nozzle0_j"
     type="fixed">
     <origin
@@ -142,5 +142,5 @@
       link="spot_boom" />
     <child
-      link="spot_nozzle3" />
+      link="spot_nozzle0" />
     <axis
       xyz="0 0 0" />
